File: mm_external_uart.kicad_sch (KiCad schematic)
At the start: 0 parts

Commit message: fin tp2
Parts:
- added C7: 0.1u, Capacitor_SMD:C_0603_1608Metric, symbol Device:C
- added C8: 2.2u, Capacitor_SMD:C_0603_1608Metric, symbol Device:C
- added J4: Conn_01x04_Pin, Connector_PinHeader_2.54mm:PinHeader_1x04_P2.54mm_Vertical, symbol Connector:Conn_01x04_Pin
- added R8: 100, Resistor_SMD:R_0603_1608Metric, symbol Device:R
Connections:
- new net: J4.4 (Pin_4), R8.2
- new net +BATT: C7.1, C8.1, J4.2 (Pin_2)
- new net GND: C7.2, C8.2, J4.1 (Pin_1)
- new net UART1_RX: J4.3 (Pin_3)
- new net UART1_TX: R8.1
Changed lines of the file:
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@@
 (kicad_sch (version 20230121) (generator eeschema)
   (paper "A4")
+  (junction (at 120.65 95.25) (diameter 0) (color 0 0 0 0)
+  )
+  (junction (at 128.27 95.25) (diameter 0) (color 0 0 0 0)
+  )
+  (junction (at 134.62 104.14) (diameter 0) (color 0 0 0 0)
+  )
+  (junction (at 128.27 104.14) (diameter 0) (color 0 0 0 0)
+  )
+  (wire (pts (xy 134.62 97.79) (xy 135.89 97.79))
+    (stroke (width 0) (type default))
+  )
+  (wire (pts (xy 134.62 90.17) (xy 135.89 90.17))
+    (stroke (width 0) (type default))
+  )
+  (wire (pts (xy 128.27 104.14) (xy 134.62 104.14))
+    (stroke (width 0) (type default))
+  )
+  (wire (pts (xy 120.65 95.25) (xy 120.65 96.52))
+    (stroke (width 0) (type default))
+  )
+  (wire (pts (xy 109.22 95.25) (xy 120.65 95.25))
+    (stroke (width 0) (type default))
+  )
+  (wire (pts (xy 128.27 95.25) (xy 135.89 95.25))
+    (stroke (width 0) (type default))
+  )
+  (wire (pts (xy 125.73 92.71) (xy 135.89 92.71))
+    (stroke (width 0) (type default))
+  )
+  (wire (pts (xy 125.73 90.17) (xy 127 90.17))
+    (stroke (width 0) (type default))
+  )
+  (wire (pts (xy 120.65 95.25) (xy 128.27 95.25))
+    (stroke (width 0) (type default))
+  )
+  (wire (pts (xy 134.62 105.41) (xy 134.62 104.14))
+    (stroke (width 0) (type default))
+  )
+  (wire (pts (xy 128.27 95.25) (xy 128.27 96.52))
+    (stroke (width 0) (type default))
+  )
+  (wire (pts (xy 120.65 104.14) (xy 128.27 104.14))
+    (stroke (width 0) (type default))
+  )
+  (wire (pts (xy 134.62 104.14) (xy 134.62 97.79))
+    (stroke (width 0) (type default))
+  )
+  (hierarchical_label "UART1_TX" (shape output) (at 125.73 90.17 180) (fields_autoplaced)
+    (effects (font (size 1.27 1.27)) (justify right))
+  )
+  (hierarchical_label "UART1_RX" (shape input) (at 125.73 92.71 180) (fields_autoplaced)
+    (effects (font (size 1.27 1.27)) (justify right))
+  )
+  (symbol (lib_id "power:+BATT") (at 109.22 95.25 0) (unit 1)
+    (in_bom yes) (on_board yes) (dnp no)
+    (property "Reference" "#PWR016" (at 109.22 99.06 0)
+      (effects (font (size 1.27 1.27)) hide)
+    )
+    (property "Value" "+BATT" (at 105.41 91.44 0)
+      (effects (font (size 1.27 1.27)) (justify left))
+    )
+    (property "Footprint" "" (at 109.22 95.25 0)
+      (effects (font (size 1.27 1.27)) hide)
+    )
+    (property "Datasheet" "" (at 109.22 95.25 0)
+      (effects (font (size 1.27 1.27)) hide)
+    )
+    (pin "1")
+    (instances
+      (project "minimouse"
+        (path "/d8fa4cba-2469-4231-847f-065b6b829f44/d17bb1c7-f68a-465e-9a17-5858ef86fc30"
+          (reference "#PWR016") (unit 1)
+        )
+      )
+    )
+  )
+  (symbol (lib_id "Device:R") (at 130.81 90.17 90) (unit 1)
+    (in_bom yes) (on_board yes) (dnp no)
+    (property "Reference" "R8" (at 130.81 85.09 90)
+      (effects (font (size 1.27 1.27)))
+    )
+    (property "Value" "100" (at 130.81 87.63 90)
+      (effects (font (size 1.27 1.27)))
+    )
+    (property "Footprint" "Resistor_SMD:R_0603_1608Metric" (at 130.81 91.948 90)
+      (effects (font (size 1.27 1.27)) hide)
+    )
+    (property "Datasheet" "~" (at 130.81 90.17 0)
+      (effects (font (size 1.27 1.27)) hide)
+    )
+    (pin "1")
+    (pin "2")
+    (instances
+      (project "minimouse"
+        (path "/d8fa4cba-2469-4231-847f-065b6b829f44/b5d7e952-00af-4b6f-924a-ee43c62726d2"
+          (reference "R8") (unit 1)
+        )
+        (path "/d8fa4cba-2469-4231-847f-065b6b829f44/d17bb1c7-f68a-465e-9a17-5858ef86fc30"
+          (reference "R21") (unit 1)
+        )
+      )
+    )
+  )
+  (symbol (lib_id "Connector:Conn_01x04_Pin") (at 140.97 95.25 180) (unit 1)
+    (in_bom yes) (on_board yes) (dnp no) (fields_autoplaced)
+    (property "Reference" "J4" (at 142.24 92.71 0)
+      (effects (font (size 1.27 1.27)) (justify right))
+    )
+    (property "Value" "Conn_01x04_Pin" (at 142.24 95.25 0)
+      (effects (font (size 1.27 1.27)) (justify right))
+    )
+    (property "Footprint" "Connector_PinHeader_2.54mm:PinHeader_1x04_P2.54mm_Vertical" (at 140.97 95.25 0)
+      (effects (font (size 1.27 1.27)) hide)
+    )
+    (property "Datasheet" "~" (at 140.97 95.25 0)
+      (effects (font (size 1.27 1.27)) hide)
+    )
+    (pin "2")
+    (pin "4")
+    (pin "1")
+    (pin "3")
+    (instances
+      (project "minimouse"
+        (path "/d8fa4cba-2469-4231-847f-065b6b829f44/d17bb1c7-f68a-465e-9a17-5858ef86fc30"
+          (reference "J4") (unit 1)
+        )
+      )
+    )
+  )
+  (symbol (lib_id "Device:C") (at 128.27 100.33 0) (unit 1)
+    (in_bom yes) (on_board yes) (dnp no)
+    (property "Reference" "C7" (at 128.27 97.79 0)
+      (effects (font (size 1.27 1.27)) (justify left))
+    )
+    (property "Value" "0.1u" (at 128.27 102.87 0)
+      (effects (font (size 1.27 1.27)) (justify left))
+    )
+    (property "Footprint" "Capacitor_SMD:C_0603_1608Metric" (at 129.2352 104.14 0)
+      (effects (font (size 1.27 1.27)) hide)
+    )
+    (property "Datasheet" "~" (at 128.27 100.33 0)
+      (effects (font (size 1.27 1.27)) hide)
+    )
+    (pin "1")
+    (pin "2")
+    (instances
+      (project "minimouse"
+        (path "/d8fa4cba-2469-4231-847f-065b6b829f44/0999fad3-9a14-4ede-b729-a71c3dbbdf8e"
+          (reference "C7") (unit 1)
+        )
+        (path "/d8fa4cba-2469-4231-847f-065b6b829f44/d17bb1c7-f68a-465e-9a17-5858ef86fc30"
+          (reference "C12") (unit 1)
+        )
+      )
+    )
+  )
+  (symbol (lib_id "Device:C") (at 120.65 100.33 0) (unit 1)
+    (in_bom yes) (on_board yes) (dnp no)
+    (property "Reference" "C8" (at 121.92 97.79 0)
+      (effects (font (size 1.27 1.27)) (justify left))
+    )
+    (property "Value" "2.2u" (at 121.92 102.87 0)
+      (effects (font (size 1.27 1.27)) (justify left))
+    )
+    (property "Footprint" "Capacitor_SMD:C_0603_1608Metric" (at 121.6152 104.14 0)
+      (effects (font (size 1.27 1.27)) hide)
+    )
+    (property "Datasheet" "~" (at 120.65 100.33 0)
+      (effects (font (size 1.27 1.27)) hide)
+    )
+    (pin "1")
+    (pin "2")
+    (instances
+      (project "minimouse"
+        (path "/d8fa4cba-2469-4231-847f-065b6b829f44/0999fad3-9a14-4ede-b729-a71c3dbbdf8e"
+          (reference "C8") (unit 1)
+        )
+        (path "/d8fa4cba-2469-4231-847f-065b6b829f44/7f113667-692a-4f4d-b16f-621d32f3f136"
+          (reference "C17") (unit 1)
+        )
+        (path "/d8fa4cba-2469-4231-847f-065b6b829f44/3975acd0-18ad-47bc-9ce1-d8c4d864aafe"
+          (reference "C18") (unit 1)
+        )
+        (path "/d8fa4cba-2469-4231-847f-065b6b829f44/d17bb1c7-f68a-465e-9a17-5858ef86fc30"
+          (reference "C19") (unit 1)
+        )
+      )
+    )
+  )
+  (symbol (lib_id "power:GND") (at 134.62 105.41 0) (unit 1)
+    (in_bom yes) (on_board yes) (dnp no) (fields_autoplaced)
+    (property "Reference" "#PWR017" (at 134.62 111.76 0)
+      (effects (font (size 1.27 1.27)) hide)
+    )
+    (property "Value" "GND" (at 134.62 110.49 0)
+      (effects (font (size 1.27 1.27)))
+    )
+    (property "Footprint" "" (at 134.62 105.41 0)
+      (effects (font (size 1.27 1.27)) hide)
+    )
+    (property "Datasheet" "" (at 134.62 105.41 0)
+      (effects (font (size 1.27 1.27)) hide)
+    )
+    (pin "1")
+    (instances
+      (project "minimouse"
+        (path "/d8fa4cba-2469-4231-847f-065b6b829f44/d17bb1c7-f68a-465e-9a17-5858ef86fc30"
+          (reference "#PWR017") (unit 1)
+        )
+      )
+    )
+  )
 )

Commit message: tp3
Parts:
- removed C7: 0.1u, Capacitor_SMD:C_0603_1608Metric, symbol Device:C
- removed C8: 2.2u, Capacitor_SMD:C_0603_1608Metric, symbol Device:C
- added C10: 2.2u, symbol Device:C
- renumbered R8 to R21
Connections:
- net UART1_RX is gone; now on an unnamed net: J4.3 (Pin_3)
- net +BATT: now also C10.1
- net GND: now also C10.2
- net at R21.2: no longer J4.4 (Pin_4)
- net UART1_TX renamed EXT_UART_TX
- new net EXT_UART_RX: J4.4 (Pin_4)
Other:
- moved on the sheet: R21
Changed lines of the file:
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@@
 (kicad_sch (version 20230121) (generator eeschema)
   (paper "A4")
-  (junction (at 120.65 95.25) (diameter 0) (color 0 0 0 0)
-  )
-  (junction (at 128.27 95.25) (diameter 0) (color 0 0 0 0)
-  )
-  (junction (at 134.62 104.14) (diameter 0) (color 0 0 0 0)
-  )
-  (junction (at 128.27 104.14) (diameter 0) (color 0 0 0 0)
-  )
   (wire (pts (xy 134.62 97.79) (xy 135.89 97.79))
     (stroke (width 0) (type default))
   )
-  (wire (pts (xy 134.62 90.17) (xy 135.89 90.17))
+  (wire (pts (xy 133.35 92.71) (xy 135.89 92.71))
     (stroke (width 0) (type default))
   )
-  (wire (pts (xy 128.27 104.14) (xy 134.62 104.14))
+  (wire (pts (xy 124.46 90.17) (xy 135.89 90.17))
     (stroke (width 0) (type default))
   )
-  (wire (pts (xy 120.65 95.25) (xy 120.65 96.52))
+  (wire (pts (xy 109.22 95.25) (xy 135.89 95.25))
     (stroke (width 0) (type default))
   )
-  (wire (pts (xy 109.22 95.25) (xy 120.65 95.25))
+  (wire (pts (xy 124.46 92.71) (xy 125.73 92.71))
     (stroke (width 0) (type default))
   )
-  (wire (pts (xy 128.27 95.25) (xy 135.89 95.25))
+  (wire (pts (xy 134.62 97.79) (xy 134.62 105.41))
     (stroke (width 0) (type default))
   )
-  (wire (pts (xy 125.73 92.71) (xy 135.89 92.71))
-    (stroke (width 0) (type default))
-  )
-  (wire (pts (xy 125.73 90.17) (xy 127 90.17))
-    (stroke (width 0) (type default))
-  )
-  (wire (pts (xy 120.65 95.25) (xy 128.27 95.25))
-    (stroke (width 0) (type default))
-  )
-  (wire (pts (xy 134.62 105.41) (xy 134.62 104.14))
-    (stroke (width 0) (type default))
-  )
-  (wire (pts (xy 128.27 95.25) (xy 128.27 96.52))
-    (stroke (width 0) (type default))
-  )
-  (wire (pts (xy 120.65 104.14) (xy 128.27 104.14))
-    (stroke (width 0) (type default))
-  )
-  (wire (pts (xy 134.62 104.14) (xy 134.62 97.79))
-    (stroke (width 0) (type default))
-  )
-  (hierarchical_label "UART1_TX" (shape output) (at 125.73 90.17 180) (fields_autoplaced)
+  (hierarchical_label "EXT_UART_TX" (shape output) (at 124.46 92.71 180) (fields_autoplaced)
     (effects (font (size 1.27 1.27)) (justify right))
   )
-  (hierarchical_label "UART1_RX" (shape input) (at 125.73 92.71 180) (fields_autoplaced)
+  (hierarchical_label "EXT_UART_RX" (shape input) (at 124.46 90.17 180) (fields_autoplaced)
     (effects (font (size 1.27 1.27)) (justify right))
+  )
+  (symbol (lib_id "power:GND") (at 173.99 85.09 0) (unit 1)
+    (in_bom yes) (on_board yes) (dnp no) (fields_autoplaced)
+    (property "Reference" "#PWR030" (at 173.99 91.44 0)
+      (effects (font (size 1.27 1.27)) hide)
+    )
+    (property "Value" "GND" (at 173.99 90.17 0)
+      (effects (font (size 1.27 1.27)))
+    )
+    (property "Footprint" "" (at 173.99 85.09 0)
+      (effects (font (size 1.27 1.27)) hide)
+    )
+    (property "Datasheet" "" (at 173.99 85.09 0)
+      (effects (font (size 1.27 1.27)) hide)
+    )
+    (pin "1")
+    (instances
+      (project "minimouse"
+        (path "/d8fa4cba-2469-4231-847f-065b6b829f44/d17bb1c7-f68a-465e-9a17-5858ef86fc30"
+          (reference "#PWR030") (unit 1)
+        )
+      )
+    )
+  )
+  (symbol (lib_id "power:+BATT") (at 173.99 77.47 0) (unit 1)
+    (in_bom yes) (on_board yes) (dnp no) (fields_autoplaced)
+    (property "Reference" "#PWR029" (at 173.99 81.28 0)
+      (effects (font (size 1.27 1.27)) hide)
+    )
+    (property "Value" "+BATT" (at 173.99 72.39 0)
+      (effects (font (size 1.27 1.27)))
+    )
+    (property "Footprint" "" (at 173.99 77.47 0)
+      (effects (font (size 1.27 1.27)) hide)
+    )
+    (property "Datasheet" "" (at 173.99 77.47 0)
+      (effects (font (size 1.27 1.27)) hide)
+    )
+    (pin "1")
+    (instances
+      (project "minimouse"
+        (path "/d8fa4cba-2469-4231-847f-065b6b829f44/d17bb1c7-f68a-465e-9a17-5858ef86fc30"
+          (reference "#PWR029") (unit 1)
+        )
+      )
+    )
+  )
+  (symbol (lib_id "Device:C") (at 173.99 81.28 0) (unit 1)
+    (in_bom yes) (on_board yes) (dnp no) (fields_autoplaced)
+    (property "Reference" "C10" (at 177.8 80.01 0)
+      (effects (font (size 1.27 1.27)) (justify left))
+    )
+    (property "Value" "2.2u" (at 177.8 82.55 0)
+      (effects (font (size 1.27 1.27)) (justify left))
+    )
+    (property "Footprint" "" (at 174.9552 85.09 0)
+      (effects (font (size 1.27 1.27)) hide)
+    )
+    (property "Datasheet" "~" (at 173.99 81.28 0)
+      (effects (font (size 1.27 1.27)) hide)
+    )
+    (pin "2")
+    (pin "1")
+    (instances
+      (project "minimouse"
+        (path "/d8fa4cba-2469-4231-847f-065b6b829f44/d17bb1c7-f68a-465e-9a17-5858ef86fc30"
+          (reference "C10") (unit 1)
+        )
+      )
+    )
   )
   (symbol (lib_id "power:+BATT") (at 109.22 95.25 0) (unit 1)
@@
     )
   )
-  (symbol (lib_id "Device:R") (at 130.81 90.17 90) (unit 1)
+  (symbol (lib_id "Device:R") (at 129.54 92.71 90) (unit 1)
     (in_bom yes) (on_board yes) (dnp no)
-    (property "Reference" "R8" (at 130.81 85.09 90)
+    (property "Reference" "R21" (at 129.54 87.63 90)
       (effects (font (size 1.27 1.27)))
     )
-    (property "Value" "100" (at 130.81 87.63 90)
+    (property "Value" "100" (at 129.54 90.17 90)
       (effects (font (size 1.27 1.27)))
     )
-    (property "Footprint" "Resistor_SMD:R_0603_1608Metric" (at 130.81 91.948 90)
+    (property "Footprint" "Resistor_SMD:R_0603_1608Metric" (at 129.54 94.488 90)
       (effects (font (size 1.27 1.27)) hide)
     )
-    (property "Datasheet" "~" (at 130.81 90.17 0)
+    (property "Datasheet" "~" (at 129.54 92.71 0)
       (effects (font (size 1.27 1.27)) hide)
     )
@@
     (instances
       (project "minimouse"
-        (path "/d8fa4cba-2469-4231-847f-065b6b829f44/b5d7e952-00af-4b6f-924a-ee43c62726d2"
-          (reference "R8") (unit 1)
-        )
         (path "/d8fa4cba-2469-4231-847f-065b6b829f44/d17bb1c7-f68a-465e-9a17-5858ef86fc30"
           (reference "R21") (unit 1)
@@
         )
       )
-    )
-  )
-  (symbol (lib_id "Device:C") (at 128.27 100.33 0) (unit 1)
-    (in_bom yes) (on_board yes) (dnp no)
-    (property "Reference" "C7" (at 128.27 97.79 0)
-      (effects (font (size 1.27 1.27)) (justify left))
-    )
-    (property "Value" "0.1u" (at 128.27 102.87 0)
-      (effects (font (size 1.27 1.27)) (justify left))
-    )
-    (property "Footprint" "Capacitor_SMD:C_0603_1608Metric" (at 129.2352 104.14 0)
-      (effects (font (size 1.27 1.27)) hide)
-    )
-    (property "Datasheet" "~" (at 128.27 100.33 0)
-      (effects (font (size 1.27 1.27)) hide)
-    )
-    (pin "1")
-    (pin "2")
-    (instances
-      (project "minimouse"
-        (path "/d8fa4cba-2469-4231-847f-065b6b829f44/0999fad3-9a14-4ede-b729-a71c3dbbdf8e"
-          (reference "C7") (unit 1)
-        )
-        (path "/d8fa4cba-2469-4231-847f-065b6b829f44/d17bb1c7-f68a-465e-9a17-5858ef86fc30"
-          (reference "C12") (unit 1)
-        )
-      )
-    )
-  )
-  (symbol (lib_id "Device:C") (at 120.65 100.33 0) (unit 1)
-    (in_bom yes) (on_board yes) (dnp no)
-    (property "Reference" "C8" (at 121.92 97.79 0)
-      (effects (font (size 1.27 1.27)) (justify left))
-    )
-    (property "Value" "2.2u" (at 121.92 102.87 0)
-      (effects (font (size 1.27 1.27)) (justify left))
-    )
-    (property "Footprint" "Capacitor_SMD:C_0603_1608Metric" (at 121.6152 104.14 0)
-      (effects (font (size 1.27 1.27)) hide)
-    )
-    (property "Datasheet" "~" (at 120.65 100.33 0)
-      (effects (font (size 1.27 1.27)) hide)
-    )
-    (pin "1")
-    (pin "2")
-    (instances
-      (project "minimouse"
-        (path "/d8fa4cba-2469-4231-847f-065b6b829f44/0999fad3-9a14-4ede-b729-a71c3dbbdf8e"
-          (reference "C8") (unit 1)
-        )
-        (path "/d8fa4cba-2469-4231-847f-065b6b829f44/7f113667-692a-4f4d-b16f-621d32f3f136"
-          (reference "C17") (unit 1)
-        )
-        (path "/d8fa4cba-2469-4231-847f-065b6b829f44/3975acd0-18ad-47bc-9ce1-d8c4d864aafe"
-          (reference "C18") (unit 1)
-        )
-        (path "/d8fa4cba-2469-4231-847f-065b6b829f44/d17bb1c7-f68a-465e-9a17-5858ef86fc30"
-          (reference "C19") (unit 1)
-        )
-      )
