File: mm_motor.kicad_sch (KiCad schematic)
At the start: 1 part, among them M1 N20_encoder

Commit message: fin tp2
Parts:
- added C7: 0.1u, Capacitor_SMD:C_0603_1608Metric, symbol Device:C
- added C8: 2.2u, Capacitor_SMD:C_0603_1608Metric, symbol Device:C
- added J2: Conn_01x06_Pin, Connector_PinHeader_2.54mm:PinHeader_1x06_P2.54mm_Vertical, symbol Connector:Conn_01x06_Pin
- added R8 (x2): 100, Resistor_SMD:R_0603_1608Metric, symbol Device:R
Connections:
- net C1: now also R8.1
- net C2: now also R8.1
- net MA: now also J2.6 (Pin_6)
- net MB: now also J2.1 (Pin_1)
- new net: J2.3 (Pin_3), R8.2
- new net: J2.4 (Pin_4), R8.2
- new net +3.3V: C7.1, C8.1, J2.2 (Pin_2)
- new net GND: C7.2, C8.2, J2.5 (Pin_5)

Commit message: tp3
Parts:
- removed C8: 2.2u, Capacitor_SMD:C_0603_1608Metric, symbol Device:C
- C7: value 0.1u -> 2.2u
- renumbered R8 to R22, R8 to R24
Connections:
- net +3.3V renamed +BATT
