File: mm_motor_control.kicad_sch (KiCad schematic)
At the start: 0 parts

Commit message: fin tp2
Parts:
- added C15: 10n, Capacitor_SMD:C_0603_1608Metric, symbol Device:C
- added C16: 22n, Capacitor_SMD:C_0603_1608Metric, symbol Device:C
- added C23: 1n, Capacitor_SMD:C_0603_1608Metric, symbol Device:C
- added C7: 0.1u, Capacitor_SMD:C_0603_1608Metric, symbol Device:C
- added C8: 2.2u, Capacitor_SMD:C_0603_1608Metric, symbol Device:C
- added R10, R11: 10k, Resistor_SMD:R_0603_1608Metric, symbol Device:R
- added R16, R20: 18k, Resistor_SMD:R_0603_1608Metric, symbol Device:R
- added R17: 1k, Resistor_SMD:R_0603_1608Metric, symbol Device:R
- added R18: 47k, Resistor_SMD:R_0603_1608Metric, symbol Device:R
- added Rsense1, Rsense2: 330m, Resistor_SMD:R_2512_6332Metric, symbol Device:R
- added U2: ~, STSPIN240:STSPIN240, symbol STSPIN240:U1
Connections:
- net EN: now also R16.1
- net FAULT: now also C15.1, R16.2, U2.13 (EN)
- net OUT_A1: now also U2.3 (OUTA1)
- net OUT_A2: now also U2.5 (OUTA2)
- net OUT_B1: now also U2.10 (OUTB1)
- net OUT_B2: now also U2.8 (OUTB2)
- net PHASE_A: now also U2.1 (PHA)
- net PHASE_B: now also U2.15 (PHB)
- net PWM_A: now also U2.2 (PWMA)
- net PWM_B: now also U2.16 (PWMB)
- net STBY/RESET: now also C23.1, R20.1, U2.14 (STBY)
- new net: C16.1, R17.1
- new net: R17.2, R18.2, U2.12 (TOFF)
- new net: Rsense2.1, U2.9 (SENSEB)
- new net: Rsense1.1, U2.4 (SENSEA)
- new net: R10.2, R11.1, U2.11 (REF)
- new net +3.3V: C7.1, C8.1, R20.2
- new net +BATT: R11.2
- new net GND: C15.2, C16.2, C23.2, C7.2, C8.2, R10.1, R18.1, Rsense1.2, Rsense2.2, U2.17 (GND), U2.7 (GND)

Commit message: tp3
Parts:
- removed C23: 1n, Capacitor_SMD:C_0603_1608Metric, symbol Device:C
- removed C7: 0.1u, Capacitor_SMD:C_0603_1608Metric, symbol Device:C
- removed R20: 18k, Resistor_SMD:R_0603_1608Metric, symbol Device:R
- C15: value 10n -> 1n
- R16: value 18k -> 10k
Connections:
- net +3.3V is gone; now on net +BATT: C8.1
Other:
- moved on the sheet: C8
