File: minimouse.kicad_pcb (KiCad board)
At the start: 2 copper layers, 90 x 85 mm, 22 parts, among them J1 Conn_ARM_JTAG_SWD_10, J5 Conn_01x02, M1 N20_encoder, M2 N20_encoder, U1 STM32F030C8Tx, U4 HC-SR04

Commit message: fin tp2
Parts:
- added C10: 0.1u, Capacitor_SMD:C_0603_1608Metric, F.Cu at (71.2, 74.1)
- added C11: 0.1u, Capacitor_SMD:C_0603_1608Metric, F.Cu at (56.5, 67.0)
- added C12: 0.1u, Capacitor_SMD:C_0603_1608Metric, F.Cu at (71.2, 87.6)
- added C13: 0.1u, Capacitor_SMD:C_0603_1608Metric, F.Cu at (71.2, 83.1)
- added C14: 0.1u, Capacitor_SMD:C_0603_1608Metric, F.Cu at (71.2, 78.6)
- added C15: 10n, Capacitor_SMD:C_0603_1608Metric, F.Cu at (53.4, 124.0)
- added C16: 22n, Capacitor_SMD:C_0603_1608Metric, F.Cu at (53.4, 126.5)
- added C17: 2.2u, Capacitor_SMD:C_0603_1608Metric, F.Cu at (65.4, 128.5)
- added C18: 2.2u, Capacitor_SMD:C_0603_1608Metric, F.Cu at (65.4, 124.0)
- added C19: 2.2u, Capacitor_SMD:C_0603_1608Metric, F.Cu at (65.4, 133.0)
- added C20: 2.2u, Capacitor_SMD:C_0603_1608Metric, F.Cu at (59.4, 133.5)
- added C21: 2.2u, Capacitor_SMD:C_0603_1608Metric, F.Cu at (59.4, 124.0)
- added C22: 2.2u, Capacitor_SMD:C_0603_1608Metric, F.Cu at (59.4, 126.5)
- added C23: 1n, Capacitor_SMD:C_0603_1608Metric, F.Cu at (73.0, 125.4)
- added C7: 0.1u, Capacitor_SMD:C_0603_1608Metric, F.Cu at (56.5, 71.6)
- added C8: 2.2u, Capacitor_SMD:C_0603_1608Metric, F.Cu at (56.5, 74.1)
- added C9: 0.1u, Capacitor_SMD:C_0603_1608Metric, F.Cu at (71.2, 71.6)
- added D1: LED, LED_SMD:LED_0603_1608Metric, F.Cu at (78.1, 79.7)
- added J2: Conn_01x06_Pin, Connector_PinHeader_2.54mm:PinHeader_1x06_P2.54mm_Vertical, F.Cu at (72.2, 100.0)
- added J3: Conn_01x06_Pin, Connector_PinHeader_2.54mm:PinHeader_1x06_P2.54mm_Vertical, F.Cu at (65.6, 100.0)
- added J4: Conn_01x04_Pin, Connector_PinHeader_2.54mm:PinHeader_1x04_P2.54mm_Vertical, F.Cu at (78.9, 100.0)
- added R10: 10k, Resistor_SMD:R_0603_1608Metric, F.Cu at (56.5, 76.6)
- added R11: 10k, Resistor_SMD:R_0603_1608Metric, F.Cu at (56.5, 79.1)
- added R12: 100, Resistor_SMD:R_0603_1608Metric, F.Cu at (56.5, 81.6)
- added R13: 100, Resistor_SMD:R_0603_1608Metric, F.Cu at (56.5, 84.1)
- added R14: 100, Resistor_SMD:R_0603_1608Metric, F.Cu at (56.5, 86.6)
- added R15: 100, Resistor_SMD:R_0603_1608Metric, F.Cu at (56.5, 89.1)
- added R16: 18k, Resistor_SMD:R_0603_1608Metric, F.Cu at (53.4, 129.0)
- added R17: 1k, Resistor_SMD:R_0603_1608Metric, F.Cu at (53.4, 131.5)
- added R18: 47k, Resistor_SMD:R_0603_1608Metric, F.Cu at (53.4, 134.0)
- added R19: 500, Resistor_SMD:R_0603_1608Metric, F.Cu at (59.4, 129.0)
- added R20: 18k, Resistor_SMD:R_0603_1608Metric, F.Cu at (73.0, 127.9)
- added R21: 100, Resistor_SMD:R_0603_1608Metric, F.Cu at (82.2, 133.0)
- added R22: 100, Resistor_SMD:R_0603_1608Metric, F.Cu at (88.2, 126.0)
- added R23: 100, Resistor_SMD:R_0603_1608Metric, F.Cu at (82.2, 126.0)
- added R24: 100, Resistor_SMD:R_0603_1608Metric, F.Cu at (88.2, 128.5)
- added R25: 100, Resistor_SMD:R_0603_1608Metric, F.Cu at (82.2, 128.5)
- added R26: 100, Resistor_SMD:R_0603_1608Metric, F.Cu at (88.2, 133.0)
- added Rsense1: 330m, Resistor_SMD:R_2512_6332Metric, F.Cu at (62.9, 72.7)
- added Rsense2: 330m, Resistor_SMD:R_2512_6332Metric, F.Cu at (62.9, 77.6)
- added U2: ~, STSPIN240:STSPIN240, F.Cu at (61.4, 82.3)
- added U3: LP5907MFX-1.2, Package_TO_SOT_SMD:SOT-23-5, F.Cu at (75.8, 72.5)
- added U4: HC-SR04, minimouse:HC-SR04, F.Cu at (87.8, 59.4)

Commit message: tp3
Parts:
- removed C10, C11, C12, C13, C14: 0.1u, Capacitor_SMD:C_0603_1608Metric
- removed C17, C18, C19: 2.2u, Capacitor_SMD:C_0603_1608Metric
- removed C23: 1n, Capacitor_SMD:C_0603_1608Metric
- removed R12, R13, R14, R15, R7: 100, Resistor_SMD:R_0603_1608Metric
- removed R20: 18k, Resistor_SMD:R_0603_1608Metric
- removed the U4 at (87.8, 59.4)
- C15: value 10n -> 1n
- C7, C9: value 0.1u -> 2.2u
- R16: value 18k -> 10k
- R19: value 500 -> 330
- moved C7 134.9 mm to (189.6, 93.6), turned to 90 degrees
- moved R19 124.7 mm to (174.7, 81.6), turned to 180 degrees
- moved C22 123.0 mm to (174.7, 83.8)
- moved C21 122.0 mm to (176.6, 90.3)
- moved J2 120.0 mm to (192.2, 97.3), turned to -90 degrees
- moved C20 113.5 mm to (154.6, 71.8)
- moved C8 111.2 mm to (165.3, 97.1), turned to -90 degrees
- moved R10 109.4 mm to (163.5, 99.6), turned to 180 degrees
- moved R11 107.7 mm to (162.7, 97.0), turned to 90 degrees
- moved R17 104.7 mm to (155.1, 106.5), turned to -90 degrees
- moved Rsense2 103.7 mm to (163.2, 103.9)
- moved R18 103.5 mm to (153.2, 106.5), turned to -90 degrees
- moved C16 103.2 mm to (154.1, 104.0), turned to 180 degrees
- moved R24 101.6 mm to (183.3, 92.8)
- moved D1 100.7 mm to (178.8, 82.4), turned to 90 degrees
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Connections:
- C7 pad 1: +3.3V -> +BATT
- C8 pad 1: +3.3V -> +BATT
- D1 pad 1: Net-(D1-K) -> GND
- D1 pad 2: +3.3V -> Net-(D1-A)
- J2 pad 2: +3.3V -> +BATT
- J3 pad 2: +3.3V -> +BATT
- J4 pad 3: /external_uart/UART1_RX -> Net-(J4-Pin_3)
- J4 pad 4: Net-(J4-Pin_4) -> /external_uart/EXT_UART_RX
- R19 pad 1: GND -> Net-(D1-A)
- R19 pad 2: Net-(D1-K) -> +3.3V
- R21 pad 1: /external_uart/UART1_TX -> /external_uart/EXT_UART_TX
- R21 pad 2: Net-(J4-Pin_4) -> Net-(J4-Pin_3)
- R8 pad 1: /mcu/UART1_TX -> /external_uart/EXT_UART_RX
- U1 pad 19: Net-(U1-PB1) -> /mcu/OUT_B1
- U1 pad 43: /mcu/UART1_RX -> /external_uart/EXT_UART_TX
- U4 pad 4: +3V3 -> +3.3V
Routing:
- net +BATT: track 0.00 -> 173.2 mm, vias 0 -> 1
- net +3.3V: track 0.00 -> 66.7 mm, vias 0 -> 2
- net /motorB/MB: track 0.00 -> 48.6 mm, vias 0 -> 2
- net /motorA/MB: track 0.00 -> 47.8 mm
- net /mcu/TIM3_CH1: track 0.00 -> 40.6 mm, vias 0 -> 2
- net /mcu/TIM3_CH2: track 0.00 -> 37.7 mm, vias 0 -> 2
- net /motorA/MA: track 0.00 -> 36.4 mm
- net /motorB/MA: track 0.00 -> 34.4 mm
- net /mcu/TIM2_CH2: track 0.00 -> 27.2 mm, vias 0 -> 2
- net /mcu/TIM2_CH1: track 0.00 -> 27.2 mm
- net Net-(U2-REF): track 0.00 -> 20.9 mm
- net /mcu/TIM15_CH1: track 0.00 -> 19.3 mm
- net /mcu/~{RESET}: track 0.00 -> 19.1 mm, vias 0 -> 2
- net /external_uart/EXT_UART_TX: track 0.00 -> 18.9 mm, vias 0 -> 2
- net /mcu/IN_B2: track 0.00 -> 18.1 mm
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- added copper zone on B.Cu, net GND

Commit message: tp3
Parts:
- moved R21 8.34 mm to (156.2, 79.1), turned to 0 degrees
- moved Rsense2 7.18 mm to (170.0, 101.6)
- moved C9 7.12 mm to (110.7, 89.7), turned to 90 degrees
- moved Rsense1 6.22 mm to (130.1, 97.7)
- moved BOOT0 4.36 mm to (152.8, 77.9)
- moved R22 3.86 mm to (180.1, 92.7)
- moved U2 3.44 mm to (147.0, 107.9)
- moved R8 3.20 mm to (156.2, 80.9), turned to 180 degrees
- moved C21 3.18 mm to (178.1, 87.5), turned to 90 degrees
- moved R10 3.14 mm to (160.8, 98.0), turned to 90 degrees
- moved R2 3.00 mm to (140.9, 95.4)
- moved R24 2.91 mm to (181.1, 90.9)
- moved J2 2.83 mm to (189.8, 95.7)
- moved C8 2.33 mm to (164.9, 94.8), turned to 90 degrees
- moved C15 2.20 mm to (150.0, 102.9)
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Routing:
- net +3.3V: track 66.7 -> 110.2 mm
- net +BATT: track 173.2 -> 206.9 mm, vias 1 -> 2
- net GND: track 0.00 -> 13.4 mm, vias 0 -> 41
- net Net-(J4-Pin_3): track 2.68 -> 14.6 mm
- net /external_uart/EXT_UART_TX: track 18.9 -> 9.25 mm, vias 2 -> 0
- net Net-(U2-SENSEB): track 13.6 -> 22.4 mm
- net /mcu/TIM15_CH1: track 19.3 -> 13.7 mm
- net /motorB/MB: track 48.6 -> 44.2 mm, vias 2 -> 0
- net /motorB/MA: track 34.4 -> 30.4 mm
- net /mcu/OUT_B0: track 11.0 -> 7.27 mm
- net Net-(U1-PA2): track 2.58 -> 6.24 mm
- net /external_uart/EXT_UART_RX: track 13.2 -> 9.72 mm
- net /mcu/OUT_A4: track 11.8 -> 8.34 mm
- net /mcu/TIM15_CH2: track 11.9 -> 8.43 mm
- net /mcu/BOOT0: track 12.5 -> 9.36 mm
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- added copper zone on F.Cu, net GND

Commit message: tp4
Routing:
- net GND: vias 41 -> 46
Changed lines of the file:
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@@
       (outputformat 1)
       (mirror false)
-      (drillshape 1)
+      (drillshape 0)
       (scaleselection 1)
-      (outputdirectory "")
+      (outputdirectory "fabrication_output/")
     )
   )
@@
     (fp_line (start 3.15 1.6) (end -3.15 1.6)
       (stroke (width 0.1) (type solid)) (layer "F.Fab"))
-    (pad "1" smd roundrect (at -2.9625 0 180) (size 1.225 3.35) (layers "F.Cu" "F.Paste" "F.Mask") (roundrect_rratio 0.204082)
+    (pad "1" smd roundrect (at -2.9625 0 180) (size 1.225 3.35) (layers "F.Cu" "F.Paste" "F.Mask") (roundrect_rratio 0.2040816327)
       (net 57 "Net-(U2-SENSEA)") (pintype "passive"))
-    (pad "2" smd roundrect (at 2.9625 0 180) (size 1.225 3.35) (layers "F.Cu" "F.Paste" "F.Mask") (roundrect_rratio 0.204082)
+    (pad "2" smd roundrect (at 2.9625 0 180) (size 1.225 3.35) (layers "F.Cu" "F.Paste" "F.Mask") (roundrect_rratio 0.2040816327)
       (net 2 "GND") (pintype "passive"))
     (model "${KICAD6_3DMODEL_DIR}/Resistor_SMD.3dshapes/R_2512_6332Metric.wrl"
@@
     (fp_line (start 3.15 1.6) (end -3.15 1.6)
       (stroke (width 0.1) (type solid)) (layer "F.Fab"))
-    (pad "1" smd roundrect (at -2.9625 0) (size 1.225 3.35) (layers "F.Cu" "F.Paste" "F.Mask") (roundrect_rratio 0.204082)
+    (pad "1" smd roundrect (at -2.9625 0) (size 1.225 3.35) (layers "F.Cu" "F.Paste" "F.Mask") (roundrect_rratio 0.2040816327)
       (net 58 "Net-(U2-SENSEB)") (pintype "passive"))
-    (pad "2" smd roundrect (at 2.9625 0) (size 1.225 3.35) (layers "F.Cu" "F.Paste" "F.Mask") (roundrect_rratio 0.204082)
+    (pad "2" smd roundrect (at 2.9625 0) (size 1.225 3.35) (layers "F.Cu" "F.Paste" "F.Mask") (roundrect_rratio 0.2040816327)
       (net 2 "GND") (pintype "passive"))
     (model "${KICAD6_3DMODEL_DIR}/Resistor_SMD.3dshapes/R_2512_6332Metric.wrl"
@@
   (via (at 154.9 85.4) (size 0.5) (drill 0.3) (layers "F.Cu" "B.Cu") (free) (net 2))
   (via (at 120.7 85.3) (size 0.5) (drill 0.3) (layers "F.Cu" "B.Cu") (free) (net 2))
+  (via (at 107.3 98.4) (size 0.5) (drill 0.3) (layers "F.Cu" "B.Cu") (free) (net 2))
   (via (at 157.4 83.4) (size 0.5) (drill 0.3) (layers "F.Cu" "B.Cu") (free) (net 2))
+  (via (at 123.7 73.6) (size 0.5) (drill 0.3) (layers "F.Cu" "B.Cu") (free) (net 2))
   (via (at 174.9 87.1125) (size 0.5) (drill 0.3) (layers "F.Cu" "B.Cu") (free) (net 2))
   (via (at 179.5 104.7) (size 0.5) (drill 0.3) (layers "F.Cu" "B.Cu") (free) (net 2))
@@
   (via (at 164.4 84.2) (size 0.5) (drill 0.3) (layers "F.Cu" "B.Cu") (free) (net 2))
   (via (at 136.3 87.8) (size 0.5) (drill 0.3) (layers "F.Cu" "B.Cu") (free) (net 2))
+  (via (at 193.4 98.5) (size 0.5) (drill 0.3) (layers "F.Cu" "B.Cu") (free) (net 2))
   (via (at 160.7 76) (size 0.5) (drill 0.3) (layers "F.Cu" "B.Cu") (free) (net 2))
   (via (at 177.5 84.8) (size 0.5) (drill 0.3) (layers "F.Cu" "B.Cu") (free) (net 2))
+  (via (at 175.5 67.7) (size 0.5) (drill 0.3) (layers "F.Cu" "B.Cu") (free) (net 2))
   (via (at 162.6 98.8) (size 0.5) (drill 0.3) (layers "F.Cu" "B.Cu") (free) (net 2))
   (via (at 138.6 94.8) (size 0.5) (drill 0.3) (layers "F.Cu" "B.Cu") (free) (net 2))
@@
   (via (at 153.6 100.1) (size 0.5) (drill 0.3) (layers "F.Cu" "B.Cu") (free) (net 2))
   (via (at 152.1 95.8) (size 0.5) (drill 0.3) (layers "F.Cu" "B.Cu") (free) (net 2))
+  (via (at 186.3 78.5) (size 0.5) (drill 0.3) (layers "F.Cu" "B.Cu") (free) (net 2))
   (via (at 183.3 93.4) (size 0.5) (drill 0.3) (layers "F.Cu" "B.Cu") (free) (net 2))
   (via (at 152.8 82.8) (size 0.5) (drill 0.3) (layers "F.Cu" "B.Cu") (free) (net 2))

Commit message: tp3
Routing:
- net /mcu/TIM2_CH2: track 27.2 -> 27.9 mm
- net GND: vias 46 -> 48
Changed lines of the file:
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@@
   (via (at 145.209751 94.060344) (size 0.5) (drill 0.3) (layers "F.Cu" "B.Cu") (free) (net 2))
   (via (at 171.7 95.2) (size 0.5) (drill 0.3) (layers "F.Cu" "B.Cu") (free) (net 2))
+  (via (at 124.5 96) (size 0.5) (drill 0.3) (layers "F.Cu" "B.Cu") (free) (net 2))
   (via (at 154.9 85.4) (size 0.5) (drill 0.3) (layers "F.Cu" "B.Cu") (free) (net 2))
   (via (at 120.7 85.3) (size 0.5) (drill 0.3) (layers "F.Cu" "B.Cu") (free) (net 2))
@@
   (via (at 193.4 98.5) (size 0.5) (drill 0.3) (layers "F.Cu" "B.Cu") (free) (net 2))
   (via (at 160.7 76) (size 0.5) (drill 0.3) (layers "F.Cu" "B.Cu") (free) (net 2))
+  (via (at 128.6 95.3) (size 0.5) (drill 0.3) (layers "F.Cu" "B.Cu") (free) (net 2))
   (via (at 177.5 84.8) (size 0.5) (drill 0.3) (layers "F.Cu" "B.Cu") (free) (net 2))
   (via (at 175.5 67.7) (size 0.5) (drill 0.3) (layers "F.Cu" "B.Cu") (free) (net 2))
@@
   (segment (start 149.1 82.125) (end 150.1 81.125) (width 0.2) (layer "F.Cu") (net 5))
   (segment (start 152.8 79) (end 152.8 77.9) (width 0.2) (layer "F.Cu") (net 5))
-  (segment (start 140.9 94.575) (end 140.9 93.7) (width 0.2) (layer "F.Cu") (net 6))
-  (segment (start 140.9 93.7) (end 142.3 92.3) (width 0.2) (layer "F.Cu") (net 6))
-  (segment (start 142.3 92.3) (end 145.6875 92.3) (width 0.2) (layer "F.Cu") (net 6))
+  (segment (start 140.9 94.4) (end 143 92.3) (width 0.2) (layer "F.Cu") (net 6))
+  (segment (start 140.9 94.575) (end 140.9 94.4) (width 0.2) (layer "F.Cu") (net 6))
+  (segment (start 143 92.3) (end 145.6875 92.3) (width 0.2) (layer "F.Cu") (net 6))
   (segment (start 140.9 101.2) (end 143.4 103.7) (width 0.2) (layer "F.Cu") (net 7))
   (segment (start 143.4 103.7) (end 143.4 106.065686) (width 0.2) (layer "F.Cu") (net 7))
@@
   (segment (start 149.45 98.3) (end 147.85 96.7) (width 0.2) (layer "B.Cu") (net 20))
   (segment (start 150.4 98.3) (end 149.45 98.3) (width 0.2) (layer "B.Cu") (net 20))
-  (segment (start 136.3 91.3) (end 132.1 87.1) (width 0.2) (layer "F.Cu") (net 21))
   (segment (start 121.1 90.6) (end 119.945 90.6) (width 0.2) (layer "F.Cu") (net 21))
-  (segment (start 145.6875 91.3) (end 136.3 91.3) (width 0.2) (layer "F.Cu") (net 21))
   (segment (start 122 88.8) (end 122 89.7) (width 0.2) (layer "F.Cu") (net 21))
+  (segment (start 145.6875 91.3) (end 136.6 91.3) (width 0.2) (layer "F.Cu") (net 21))
+  (segment (start 136.6 91.3) (end 132.4 87.1) (width 0.2) (layer "F.Cu") (net 21))
+  (segment (start 132.4 87.1) (end 123.3 87.1) (width 0.2) (layer "F.Cu") (net 21))
   (segment (start 122 89.7) (end 121.1 90.6) (width 0.2) (layer "F.Cu") (net 21))
-  (segment (start 132.1 87.1) (end 123.3 87.1) (width 0.2) (layer "F.Cu") (net 21))
   (via (at 122 88.8) (size 0.5) (drill 0.3) (layers "F.Cu" "B.Cu") (net 21))
   (via (at 123.3 87.1) (size 0.5) (drill 0.3) (layers "F.Cu" "B.Cu") (net 21))
@@
   (segment (start 149.8 97.5) (end 151.1 97.5) (width 0.2) (layer "B.Cu") (net 22))
   (segment (start 131.7 88.1) (end 120.045 88.1) (width 0.2) (layer "F.Cu") (net 23))
-  (segment (start 145.6875 91.8) (end 135.4 91.8) (width 0.2) (layer "F.Cu") (net 23))
-  (segment (start 135.4 91.8) (end 131.7 88.1) (width 0.2) (layer "F.Cu") (net 23))
+  (segment (start 136.3 92.7) (end 131.7 88.1) (width 0.2) (layer "F.Cu") (net 23))
+  (segment (start 145.6875 91.8) (end 142.5 91.8) (width 0.2) (layer "F.Cu") (net 23))
+  (segment (start 141.6 92.7) (end 136.3 92.7) (width 0.2) (layer "F.Cu") (net 23))
+  (segment (start 142.5 91.8) (end 141.6 92.7) (width 0.2) (layer "F.Cu") (net 23))
   (segment (start 148.6 78.7) (end 148.6 85.3875) (width 0.2) (layer "F.Cu") (net 24))
   (segment (start 151.3 73.425) (end 151.3 76) (width 0.2) (layer "F.Cu") (net 24))

Commit message: tp5
Parts:
- added C11: 2.2uF, Capacitor_SMD:C_0603_1608Metric, F.Cu at (170.7, 84.6)
- added D2: LED, LED_SMD:LED_0603_1608Metric, F.Cu at (150.8, 75.8)
- added D3: BZT52Bxx, Diode_SMD:D_SOD-123F, F.Cu at (143.5, 133.9)
- added D4: LED, LED_SMD:LED_0603_1608Metric, F.Cu at (148.6, 74.3)
- added Q2: PMOS, Package_TO_SOT_SMD:SOT-23-3, F.Cu at (143.1, 137.6)
- added R12: 300, Resistor_SMD:R_0603_1608Metric, F.Cu at (155.4, 75.8)
- added R13: 300, Resistor_SMD:R_0603_1608Metric, F.Cu at (151.9, 74.2)
- added R14: 100, Resistor_SMD:R_0603_1608Metric, F.Cu at (156.5, 82.5)
- added R7: 100k, Resistor_SMD:R_0603_1608Metric, F.Cu at (149.7, 132.2)
- added SW1: SW_Push, Button_Switch_SMD:SW_Push_SPST_NO_Alps_SKRK, F.Cu at (167.1, 85.7)
- moved R26 6.80 mm to (145.1, 75.4)
- moved C20 1.62 mm to (153.1, 72.4), turned to 180 degrees
Connections:
- C20 pad 1: +3.3V -> +BATT
- J5 pad 2: +BATT -> Net-(J5-Pin_2)
- U1 pad 7: /mcu/~{RESET} -> Net-(U1-NRST)
- U4 pad 4: +3.3V -> +BATT
Routing:
- net +BATT: track 206.9 -> 243.0 mm
- net Net-(U1-NRST): track 0.00 -> 15.0 mm, vias 0 -> 2
- net unconnected-(D4-K-Pad1): track 0.00 -> 12.3 mm, vias 0 -> 2
- net unconnected-(D2-K-Pad1): track 0.00 -> 11.0 mm, vias 0 -> 2
- net Net-(U4-ECHO): track 2.66 -> 10.4 mm
- net Net-(D3-A): track 0.00 -> 7.76 mm
- net Net-(J5-Pin_2): track 0.00 -> 6.70 mm
- net /mcu/OUT_B9: track 12.1 -> 18.5 mm
- net /mcu/~{RESET}: track 19.1 -> 14.8 mm, vias 2 -> 1
- net Net-(D2-A): track 0.00 -> 2.99 mm
- net /mcu/TIM8_CH2: track 13.1 -> 11.1 mm
- net Net-(D4-A): track 0.00 -> 1.73 mm
- net +3.3V: track 110.2 -> 109.0 mm
- net GND: vias 48 -> 54
