File: mm_power.kicad_sch (KiCad schematic)
At the start: 1 part, among them J5 Conn_01x02

Commit message: fin tp2
Parts:
- added C7 (x2): 0.1u, Capacitor_SMD:C_0603_1608Metric, symbol Device:C
- added C8 (x2): 2.2u, Capacitor_SMD:C_0603_1608Metric, symbol Device:C
- added D1: LED, LED_SMD:LED_0603_1608Metric, symbol Device:LED
- added R18: 500, Resistor_SMD:R_0603_1608Metric, symbol Device:R
- added U3: LP5907MFX-1.2, Package_TO_SOT_SMD:SOT-23-5, symbol Regulator_Linear:LP5907MFX-1.2
Connections:
- net +BATT: now also C7.1, C8.1, U3.1 (IN), U3.3 (EN)
- net GND: now also C7.2, C7.2, C8.2, C8.2, R18.1, U3.2 (GND)
- new net: D1.1 (K), R18.2
- new net +3.3V: C7.1, C8.1, D1.2 (A), U3.5 (OUT)

Commit message: tp3
Parts:
- removed C7 (x2): 0.1u, Capacitor_SMD:C_0603_1608Metric, symbol Device:C
- R19: renamed from R18; value 500 -> 330
- renumbered C8 to C21, C8 to C22
Connections:
- net +3.3V: now also R19.2; no longer D1.2 (A)
- net GND: now also D1.1 (K); no longer R19.1
- new net: D1.2 (A), R19.1
Other:
- moved on the sheet: C21, D1, R19

Commit message: tp5
Parts:
- added D3: BZT52Bxx, Diode_SMD:D_SOD-123F, symbol Diode:BZT52Bxx
- added Q2: PMOS, Package_TO_SOT_SMD:SOT-23-3, symbol Simulation_SPICE:PMOS
- added R7: 100k, Resistor_SMD:R_0603_1608Metric, symbol Device:R
Connections:
- net +BATT: now also D3.1 (K), Q2.3 (S); no longer J5.2 (Pin_2)
- net GND: now also R7.1
- new net: D3.2 (A), Q2.2 (G), R7.2
- new net: J5.2 (Pin_2), Q2.1 (D)
Other:
- moved on the sheet: J5
Changed lines of the file:
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@@
 (kicad_sch (version 20230121) (generator eeschema)
   (paper "A4")
+  (junction (at 151.13 93.98) (diameter 0) (color 0 0 0 0)
+  )
+  (junction (at 114.3 82.55) (diameter 0) (color 0 0 0 0)
+  )
+  (junction (at 86.36 99.06) (diameter 0) (color 0 0 0 0)
+  )
   (junction (at 86.36 82.55) (diameter 0) (color 0 0 0 0)
   )
-  (junction (at 151.13 93.98) (diameter 0) (color 0 0 0 0)
-  )
-  (junction (at 114.3 82.55) (diameter 0) (color 0 0 0 0)
-  )
-  (junction (at 86.36 93.98) (diameter 0) (color 0 0 0 0)
+  (junction (at 76.2 82.55) (diameter 0) (color 0 0 0 0)
+  )
+  (junction (at 66.04 90.17) (diameter 0) (color 0 0 0 0)
+  )
+  (junction (at 66.04 99.06) (diameter 0) (color 0 0 0 0)
   )
   (junction (at 151.13 82.55) (diameter 0) (color 0 0 0 0)
@@
   (junction (at 95.25 82.55) (diameter 0) (color 0 0 0 0)
   )
-  (wire (pts (xy 86.36 90.17) (xy 86.36 93.98))
+  (wire (pts (xy 86.36 93.98) (xy 86.36 99.06))
+    (stroke (width 0) (type default))
+  )
+  (wire (pts (xy 71.12 82.55) (xy 76.2 82.55))
     (stroke (width 0) (type default))
   )
@@
     (stroke (width 0) (type default))
   )
+  (wire (pts (xy 66.04 90.17) (xy 66.04 91.44))
+    (stroke (width 0) (type default))
+  )
   (wire (pts (xy 95.25 82.55) (xy 86.36 82.55))
     (stroke (width 0) (type default))
@@
     (stroke (width 0) (type default))
   )
+  (wire (pts (xy 58.42 99.06) (xy 66.04 99.06))
+    (stroke (width 0) (type default))
+  )
   (wire (pts (xy 114.3 93.98) (xy 133.35 93.98))
     (stroke (width 0) (type default))
   )
+  (wire (pts (xy 53.34 88.9) (xy 53.34 82.55))
+    (stroke (width 0) (type default))
+  )
   (wire (pts (xy 133.35 93.98) (xy 151.13 93.98))
     (stroke (width 0) (type default))
@@
     (stroke (width 0) (type default))
   )
-  (wire (pts (xy 80.01 87.63) (xy 86.36 87.63))
+  (wire (pts (xy 76.2 82.55) (xy 86.36 82.55))
     (stroke (width 0) (type default))
   )
@@
     (stroke (width 0) (type default))
   )
+  (wire (pts (xy 66.04 90.17) (xy 76.2 90.17))
+    (stroke (width 0) (type default))
+  )
   (wire (pts (xy 114.3 93.98) (xy 114.3 91.44))
     (stroke (width 0) (type default))
   )
+  (wire (pts (xy 53.34 91.44) (xy 58.42 91.44))
+    (stroke (width 0) (type default))
+  )
   (wire (pts (xy 151.13 82.55) (xy 151.13 83.82))
     (stroke (width 0) (type default))
@@
     (stroke (width 0) (type default))
   )
+  (wire (pts (xy 58.42 91.44) (xy 58.42 99.06))
+    (stroke (width 0) (type default))
+  )
+  (wire (pts (xy 66.04 99.06) (xy 86.36 99.06))
+    (stroke (width 0) (type default))
+  )
   (wire (pts (xy 123.19 82.55) (xy 125.73 82.55))
     (stroke (width 0) (type default))
@@
     (stroke (width 0) (type default))
   )
-  (wire (pts (xy 86.36 82.55) (xy 86.36 87.63))
-    (stroke (width 0) (type default))
-  )
   (wire (pts (xy 140.97 82.55) (xy 151.13 82.55))
     (stroke (width 0) (type default))
@@
     (stroke (width 0) (type default))
   )
+  (wire (pts (xy 53.34 82.55) (xy 60.96 82.55))
+    (stroke (width 0) (type default))
+  )
   (wire (pts (xy 123.19 85.09) (xy 123.19 82.55))
     (stroke (width 0) (type default))
@@
   )
   (wire (pts (xy 151.13 76.2) (xy 161.29 76.2))
-    (stroke (width 0) (type default))
-  )
-  (wire (pts (xy 86.36 93.98) (xy 86.36 99.06))
-    (stroke (width 0) (type default))
-  )
-  (wire (pts (xy 80.01 90.17) (xy 86.36 90.17))
     (stroke (width 0) (type default))
   )
@@
     )
   )
+  (symbol (lib_id "Diode:BZT52Bxx") (at 76.2 86.36 270) (unit 1)
+    (in_bom yes) (on_board yes) (dnp no) (fields_autoplaced)
+    (property "Reference" "D3" (at 78.74 85.09 90)
+      (effects (font (size 1.27 1.27)) (justify left))
+    )
+    (property "Value" "BZT52Bxx" (at 78.74 87.63 90)
+      (effects (font (size 1.27 1.27)) (justify left))
+    )
+    (property "Footprint" "Diode_SMD:D_SOD-123F" (at 71.755 86.36 0)
+      (effects (font (size 1.27 1.27)) hide)
+    )
+    (property "Datasheet" "https://diotec.com/tl_files/diotec/files/pdf/datasheets/bzt52b2v4.pdf" (at 76.2 86.36 0)
+      (effects (font (size 1.27 1.27)) hide)
+    )
+    (pin "1")
+    (pin "2")
+    (instances
+      (project "minimouse"
+        (path "/d8fa4cba-2469-4231-847f-065b6b829f44/3f9b0845-5778-418c-a7a8-03da2392145e"
+          (reference "D3") (unit 1)
+        )
+      )
+    )
+  )
+  (symbol (lib_id "Simulation_SPICE:PMOS") (at 66.04 85.09 90) (unit 1)
+    (in_bom yes) (on_board yes) (dnp no) (fields_autoplaced)
+    (property "Reference" "Q2" (at 66.04 76.2 90)
+      (effects (font (size 1.27 1.27)))
+    )
+    (property "Value" "PMOS" (at 66.04 78.74 90)
+      (effects (font (size 1.27 1.27)))
+    )
+    (property "Footprint" "Package_TO_SOT_SMD:SOT-23-3" (at 63.5 80.01 0)
+      (effects (font (size 1.27 1.27)) hide)
+    )
+    (property "Datasheet" "https://ngspice.sourceforge.io/docs/ngspice-manual.pdf" (at 78.74 85.09 0)
+      (effects (font (size 1.27 1.27)) hide)
+    )
+    (property "Sim.Device" "PMOS" (at 83.185 85.09 0)
+      (effects (font (size 1.27 1.27)) hide)
+    )
+    (property "Sim.Type" "VDMOS" (at 85.09 85.09 0)
+      (effects (font (size 1.27 1.27)) hide)
+    )
+    (property "Sim.Pins" "1=D 2=G 3=S" (at 81.28 85.09 0)
+      (effects (font (size 1.27 1.27)) hide)
+    )
+    (pin "2")
+    (pin "1")
+    (pin "3")
+    (instances
+      (project "minimouse"
+        (path "/d8fa4cba-2469-4231-847f-065b6b829f44/3f9b0845-5778-418c-a7a8-03da2392145e"
+          (reference "Q2") (unit 1)
+        )
+      )
+    )
+  )
   (symbol (lib_id "Device:R") (at 161.29 80.01 180) (unit 1)
     (in_bom yes) (on_board yes) (dnp no)
@@
     )
   )
+  (symbol (lib_id "Device:R") (at 66.04 95.25 180) (unit 1)
+    (in_bom yes) (on_board yes) (dnp no)
+    (property "Reference" "R7" (at 69.85 93.98 0)
+      (effects (font (size 1.27 1.27)))
+    )
+    (property "Value" "100k" (at 69.85 96.52 0)
+      (effects (font (size 1.27 1.27)))
+    )
+    (property "Footprint" "Resistor_SMD:R_0603_1608Metric" (at 67.818 95.25 90)
+      (effects (font (size 1.27 1.27)) hide)
+    )
+    (property "Datasheet" "~" (at 66.04 95.25 0)
+      (effects (font (size 1.27 1.27)) hide)
+    )
+    (pin "1")
+    (pin "2")
+    (instances
+      (project "minimouse"
+        (path "/d8fa4cba-2469-4231-847f-065b6b829f44/3f9b0845-5778-418c-a7a8-03da2392145e"
+          (reference "R7") (unit 1)
+        )
+      )
+    )
+  )
   (symbol (lib_id "Regulator_Linear:LP5907MFX-1.2") (at 133.35 85.09 0) (unit 1)
     (in_bom yes) (on_board yes) (dnp no) (fields_autoplaced)
@@
     )
   )
-  (symbol (lib_id "Connector_Generic:Conn_01x02") (at 74.93 90.17 180) (unit 1)
-    (in_bom yes) (on_board yes) (dnp no) (fields_autoplaced)
-    (property "Reference" "J5" (at 74.93 81.28 0)
-      (effects (font (size 1.27 1.27)))
-    )
-    (property "Value" "Conn_01x02" (at 74.93 83.82 0)
-      (effects (font (size 1.27 1.27)))
-    )
-    (property "Footprint" "Connector_PinHeader_2.54mm:PinHeader_1x02_P2.54mm_Vertical" (at 74.93 90.17 0)
-      (effects (font (size 1.27 1.27)) hide)
-    )
-    (property "Datasheet" "~" (at 74.93 90.17 0)
-      (effects (font (size 1.27 1.27)) hide)
-    )
+  (symbol (lib_id "Connector_Generic:Conn_01x02") (at 48.26 91.44 180) (unit 1)
+    (in_bom yes) (on_board yes) (dnp no) (fields_autoplaced)
+    (property "Reference" "J5" (at 48.26 82.55 0)
+      (effects (font (size 1.27 1.27)))
+    )
+    (property "Value" "Conn_01x02" (at 48.26 85.09 0)
+      (effects (font (size 1.27 1.27)))
+    )
+    (property "Footprint" "Connector_PinHeader_2.54mm:PinHeader_1x02_P2.54mm_Vertical" (at 48.26 91.44 0)
+      (effects (font (size 1.27 1.27)) hide)
+    )
+    (property "Datasheet" "~" (at 48.26 91.44 0)
+      (effects (font (size 1.27 1.27)) hide)
+    )
